File: CyberBadge.kicad_pcb (KiCad board)
At the start: 2 copper layers, 112.5 x 41.5 mm, 569 parts, among them J1 USB_C_Receptacle_USB2.0, J2 BAT_CONN, J3 Lichtenprog_conn, Q1 SS8050-G, Q2 SS8050-G, Q3 FS8205A, Q4 AO3401A, SW1 B2, SW2 B1/BOOT, SW3 SW_SPDT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

Commit message: most of routing
Parts:
- added C1: 22uF/handsolder, Capacitor_SMD:C_0805_2012Metric_Pad1.18x1.45mm_HandSolder, B.Cu at (113.5, 62.0)
- added C2: 22uF/handsolder, Capacitor_SMD:C_0805_2012Metric_Pad1.18x1.45mm_HandSolder, B.Cu at (118.5, 54.0)
- added C3: 22uF/handsolder, Capacitor_SMD:C_0805_2012Metric_Pad1.18x1.45mm_HandSolder, B.Cu at (118.5, 57.0)
- added C4: 22uF/handsolder, Capacitor_SMD:C_0805_2012Metric_Pad1.18x1.45mm_HandSolder, B.Cu at (123.3, 54.0)
- added SW5: B2, Button_Switch_SMD:SW_SPST_TL3342, F.Cu at (156.5, 70.0)
- C5: value 4.7u -> 22uF/handsolder; footprint Capacitor_SMD:C_0402_1005Metric -> Capacitor_SMD:C_0805_2012Metric_Pad1.18x1.45mm_HandSolder
- moved R21 7.32 mm to (101.5, 105.2), turned to 180 degrees
- moved R7 4.74 mm to (88.0, 102.2), turned to -90 degrees
- moved C6 4.68 mm to (91.2, 105.2)
- moved R16 3.82 mm to (125.0, 105.2), turned to 180 degrees
- moved R1 3.25 mm to (121.2, 105.8)
- moved R15 2.85 mm to (112.1, 72.2)
- moved R2 2.80 mm to (112.1, 69.4)
- moved Q4 2.75 mm to (122.2, 103.5)
- moved R12 2.32 mm to (83.0, 104.2)
- moved R8 2.16 mm to (88.0, 104.1), turned to 90 degrees
- moved SW1 2.00 mm to (176.5, 70.0)
- moved C5 1.56 mm to (103.3, 75.2), turned to 90 degrees
- moved R19 1.00 mm to (109.5, 105.1)
- moved SW2 1.00 mm to (166.5, 70.0)
- moved C180 0.91 mm to (111.1, 105.1)
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Connections:
- J2 pad 1: Net-(F1-Pad2) -> Net-(C180-Pad2)
- J2 pad 2: Net-(C180-Pad2) -> Net-(F1-Pad2)
- Q2 pad 2: Net-(Q2-Pad2) -> /PROG_DTR
- R9 pad 1: Net-(Q2-Pad2) -> /PROG_DTR
Routing:
- net /LIPO_PRE_MOSFET: track 3.26 -> 45.0 mm, vias 0 -> 1
- net GND: track 582.2 -> 613.1 mm, vias 10 -> 30
- net Net-(C180-Pad2): track 0.00 -> 24.5 mm, vias 0 -> 1
- net +4V: track 567.2 -> 591.2 mm, vias 1 -> 23
- net +3.3V: track 0.00 -> 18.9 mm, vias 0 -> 4
- net /PROG_DTR: track 0.00 -> 18.6 mm, vias 0 -> 1
- net /ESP_EN: track 42.2 -> 55.3 mm, vias 0 -> 1
- net /PROG_RTS: track 0.00 -> 11.8 mm, vias 0 -> 1
- net Net-(Q1-Pad1): track 0.00 -> 10.6 mm, vias 0 -> 2
- net Net-(Q3-Pad5): track 0.00 -> 9.67 mm
- net Net-(Q4-Pad1): track 52.6 -> 59.7 mm
- net Net-(R16-Pad2): track 0.00 -> 6.94 mm, vias 0 -> 2
- net Net-(Q3-Pad4): track 0.00 -> 5.83 mm, vias 0 -> 2
- net Net-(F1-Pad2): track 0.00 -> 4.56 mm
- net Net-(C180-Pad1): track 0.00 -> 3.82 mm
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- added copper zone on B.Cu, net +3.3V
- added copper zone on B.Cu, net +4V
Other:
- outline, holes or cut-outs redrawn
- board text added: "+"
- board text added: "-"
- board text added: "BATTERY T_SENSE"
- board text added: "BOARD ON/OFF"
- board text added: "DOUT"
- board text added: "FUSE"
- board text added: "GND"
- board text added: "RST BUTTON"
- board text added: "VDD"

Commit message: blah blah routing planes
Parts:
- added C269: 100n, Capacitor_SMD:C_0201_0603Metric, F.Cu at (171.5, 69.7)
- added C270: 100n, Capacitor_SMD:C_0201_0603Metric, F.Cu at (161.5, 69.8)
- added C271: 100n, Capacitor_SMD:C_0201_0603Metric, F.Cu at (123.7, 69.8)
- added R10: 10k, Resistor_SMD:R_0201_0603Metric, F.Cu at (122.8, 69.8)
- added R3: 10k, Resistor_SMD:R_0201_0603Metric, F.Cu at (121.0, 69.8)
- added R6: 10k, Resistor_SMD:R_0201_0603Metric, F.Cu at (121.8, 69.8)
- moved SW1 10.0 mm to (166.5, 70.0)
- moved SW2 10.0 mm to (176.5, 70.0)
Connections:
- SW1 pad 2: unconnected-(SW1-Pad2) -> /ESP_B2
- SW5 pad 2: unconnected-(SW5-Pad2) -> /ESP_B3
- U3 pad 14: unconnected-(U3-Pad14) -> /ESP_B2
- U3 pad 16: unconnected-(U3-Pad16) -> /ESP_B3
- U3 pad 23: unconnected-(U3-Pad23) -> /LIPO_VMEAS
Routing:
- net /ESP_B2: track 0.00 -> 98.0 mm, vias 0 -> 1
- net /ESP_B3: track 0.00 -> 83.3 mm, vias 0 -> 1
- net unconnected-(SW1-Pad2): track 80.2 -> 0.00 mm, vias 2 -> 0
- net /LIPO_VMEAS: track 0.00 -> 60.1 mm, vias 0 -> 1
- net GND: track 613.1 -> 644.1 mm, vias 30 -> 48
- net /ESP_BOOT: track 151.4 -> 138.5 mm, vias 4 -> 3
- net /ESP_EN: track 55.3 -> 46.4 mm
- net +4V: track 591.2 -> 593.7 mm, vias 23 -> 43
- net Net-(R10-Pad1): track 0.00 -> 0.91 mm
