File: CyberBadge.kicad_sch (KiCad schematic)
At the start: 44 parts, among them J1 USB_C_Receptacle_USB2.0, J2 BAT_CONN, Q1 MMBT3904, Q2 MMBT3904, SW1 B_RST, SW2 B1/BOOT, U1 USBLC6-2SC6, U2 CP2102N-A01-GQFN28, U3 ESP32-WROOM-32, U4 SPX3819M5-L-3-3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

Commit message: i forgor
Parts:
- added C180: 100n, Capacitor_SMD:C_0201_0603Metric, symbol Device:C_Small
- added Q3: FS8205A, Package_SO:TSSOP-8_4.4x3mm_P0.65mm, symbol LiPo_protection:FS8205A
- added R19: 200, Resistor_SMD:R_0201_0603Metric, symbol Device:R_Small
- added R20: 1k, Resistor_SMD:R_0201_0603Metric, symbol Device:R_Small
- added R21: 10k, Resistor_SMD:R_0201_0603Metric, symbol Device:R_Small
- added U6: DW01x, Package_TO_SOT_SMD:SOT-23-6, symbol LiPo_protection:DW01x
Connections:
- net GND: now also Q3.2 (S1), Q3.3 (S1), R20.1, R21.2
- new net: C180.1, R19.2, U6.5 (VCC)
- new net: C180.2, Q3.6 (S2), Q3.7 (S2), R21.1, U6.6 (GND)
- new net: Q3.5 (G2), U6.1 (OD)
- new net: R20.2, U6.2 (CS)
- new net: Q3.4 (G1), U6.3 (OC)
- new net: Q3.1 (D12), Q3.8 (D12)
- no-connect marks 26 -> 27
Other:
- note added: "add curr meas! ->"

Commit message: change pixel count
Parts:
- added J3: Lichtenprog_conn, Critbit_lib:Lichtenprog, symbol Critbit_lib:Lichtenprog_conn
- added SW3: SW_SPST, symbol Switch:SW_SPST
- Q1, Q2: value MMBT3904 -> SS8050-G
Connections:
- net +4V: now also SW3.2 (B); no longer R13.1
- net GND: now also R13.2, J3.6 (GND), J3.7 (GND); no longer J2.2 (Pin_2)
- net PROG_DTR: now also J3.3 (DTR)
- net PROG_RTS: now also J3.2 (RTS)
- net VBUS: now also J3.8 (5V)
- net PROG_RX: now reaches U2.25 (RXD)
- net PROG_RX: now also J3.4 (PROG_RX)
- net PROG_TX: now reaches U2.26 (TXD)
- net PROG_TX: now also J3.5 (PROG_TX)
- net at C10.1, J2.1 (Pin_1), U5.2 (BAT)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: now also R19.1
- net at U4.3 (EN): now also R13.1, SW3.1 (A); no longer R13.2
- net at C180.2, Q3.6 (S2), Q3.7 (S2)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: now also J2.2 (Pin_2)
- no-connect marks 27 -> 28
Other:
- added sheet WS_2columns12 (WS_2columns.kicad_sch)
- added sheet WS_2columns13 (WS_2columns.kicad_sch)
- added sheet WS_2columns14 (WS_2columns.kicad_sch)
- added sheet WS_2columns15 (WS_2columns.kicad_sch)
- note added: "TODO sprawdzić jakie CP jest w HSie"
- note added: "TODO sprawdzić tranzystory"
- moved on the sheet: C10, C179, C180, C7, C8, C9, D3, D4, J2, Q3, R13, R14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

Commit message: commit before replicatelayout
Parts:
- removed C1, C4: 100n, Capacitor_SMD:C_0201_0603Metric, symbol Device:C_Small
- removed C2, C3: 4.7u, Capacitor_SMD:C_0402_1005Metric, symbol Device:C_Small
- removed D2: LED, LED_SMD:LED_0402_1005Metric, symbol Device:LED
- removed R10, R11, R3: 2k, Resistor_SMD:R_0201_0603Metric, symbol Device:R_Small
- removed R13, R6: 10k, Resistor_SMD:R_0201_0603Metric, symbol Device:R_Small
- removed SW3: SW_SPST, symbol Switch:SW_SPST
- removed U1: USBLC6-2SC6, Package_TO_SOT_SMD:SOT-23-6, symbol Critbit_lib:USBLC6-2SC6
- removed U2: CP2102N-A01-GQFN28, Package_DFN_QFN:QFN-28-1EP_5x5mm_P0.5mm_EP3.35x3.35mm, symbol Interface_USB:CP2102N-A01-GQFN28
- added F1: 3A/slowblow, Fuse:Fuse_0603_1608Metric_Pad1.05x0.95mm_HandSolder, symbol Device:Fuse
- added H1, H2, H3, H4: SCRHOLE, MountingHole:MountingHole_3.2mm_M3, symbol Mechanical:MountingHole_Pad
- added Q4: AO3401A, Package_TO_SOT_SMD:SOT-23, symbol Transistor_FET:AO3401A
- added SW3: SW_SPDT, Button_Switch_SMD:SW_SPDT_PCM12, symbol Switch:SW_SPDT
- added SW4: RST, Button_Switch_SMD:SW_SPST_FSMSM, symbol Switch:SW_Push
- D1: LCSC C72043 -> (none)
- SW1: value B_RST -> B2
Connections:
- net RXD is gone; now on net PROG_TX: U3.34 (RXD0/IO3)
- net TXD is gone; now on net PROG_RX: U3.35 (TXD0/IO1)
- net +3.3V: now also C179.1, U4.5 (OUT)
- net +4V: now also D1.2 (A), U4.3 (EN), Q4.3 (D); no longer C8.1, D3.2 (A), D4.2 (A), U5.10 (OUT), U5.11 (OUT)
- net ESP_EN: now also SW4.2; no longer SW1.2
- net GND: now also R2.1, H1.1, H2.1, H3.1, H4.1, SW3.3 (C), SW4.1
- net PROG_DTR: no longer Q2.2 (E), R9.1
- net VBUS: no longer R1.1
- net at D1.1 (K): now also R2.2
- net LIPO_PRE_MOSFET: now reaches R1.2
- net LIPO_PRE_MOSFET: now also C8.1, D3.2 (A), D4.2 (A), U5.10 (OUT), U5.11 (OUT), Q4.2 (S); no longer R2.1
- net at C10.1, U5.2 (BAT), U5.3 (BAT): now also F1.1; no longer J2.1 (Pin_1), R19.1
- net at J1.A6 (D+): no longer J1.B6 (D+)
- net at J1.A7 (D-): no longer J1.B7 (D-)
- new net: Q4.1 (G), R1.1, SW3.2 (B)
- new net: F1.2, J2.1 (Pin_1), R19.1
- new net: Q2.2 (E), R9.1
- no-connect marks 28 -> 19
Other:
- note added: "8x32 WS2812 mini Imax: 200mA + 5mA*256 = 1500mA Iavg = 5mA* 256*(1/3)*(1/5)*(1/4) = ~25mA"
- note removed: "TODO sprawdzić jakie CP jest w HSie"
- moved on the sheet: C179, C5, C6, C9, J1, J3, Q1, Q2, R12, R4, R5, R7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

Commit message: routing and shape definiton in progress
Parts:
- added TP1, TP2, TP3: WS_IN, TestPoint:TestPoint_Pad_D1.5mm, symbol Connector:TestPoint
Connections:
- net +4V: now also TP1.1; no longer U5.5 (EN2)
- net GND: now also TP3.1
- net LIPO_PRE_MOSFET: now also U5.5 (EN2)
- net WS_OUT: now reaches U3.31 (IO19)
- net WS_OUT: now also TP2.1
Changed lines of the file:
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@@
     (stroke (width 0) (type default) (color 0 0 0 0))
   )
+  (wire (pts (xy 187.96 74.93) (xy 210.82 74.93))
+    (stroke (width 0) (type default) (color 0 0 0 0))
+  )
   (wire (pts (xy 308.61 209.55) (xy 308.61 213.36))
     (stroke (width 0) (type default) (color 0 0 0 0))
@@
     (stroke (width 0) (type default) (color 0 0 0 0))
   )
+  (wire (pts (xy 233.68 106.68) (xy 243.84 106.68))
+    (stroke (width 0) (type default) (color 0 0 0 0))
+  )
   (wire (pts (xy 187.96 49.53) (xy 193.04 49.53))
     (stroke (width 0) (type default) (color 0 0 0 0))
@@
     (stroke (width 0) (type default) (color 0 0 0 0))
   )
+  (wire (pts (xy 236.22 111.76) (xy 236.22 109.22))
+    (stroke (width 0) (type default) (color 0 0 0 0))
+  )
+  (wire (pts (xy 236.22 104.14) (xy 243.84 104.14))
+    (stroke (width 0) (type default) (color 0 0 0 0))
+  )
   (wire (pts (xy 148.59 41.91) (xy 140.97 41.91))
     (stroke (width 0) (type default) (color 0 0 0 0))
@@
     (stroke (width 0) (type default) (color 0 0 0 0))
   )
+  (wire (pts (xy 236.22 102.87) (xy 236.22 104.14))
+    (stroke (width 0) (type default) (color 0 0 0 0))
+  )
   (wire (pts (xy 176.53 208.28) (xy 179.07 208.28))
     (stroke (width 0) (type default) (color 0 0 0 0))
   )
+  (wire (pts (xy 306.07 167.64) (xy 311.15 167.64))
+    (stroke (width 0) (type default) (color 0 0 0 0))
+  )
   (wire (pts (xy 331.47 187.96) (xy 328.93 187.96))
     (stroke (width 0) (type default) (color 0 0 0 0))
@@
     (stroke (width 0) (type default) (color 0 0 0 0))
   )
+  (wire (pts (xy 236.22 109.22) (xy 243.84 109.22))
+    (stroke (width 0) (type default) (color 0 0 0 0))
+  )
   (wire (pts (xy 372.11 213.36) (xy 369.57 213.36))
     (stroke (width 0) (type default) (color 0 0 0 0))
@@
     (effects (font (size 1.27 1.27)) (justify left bottom))
   )
+  (label "WS_OUT" (at 210.82 74.93 0)
+    (effects (font (size 1.27 1.27)) (justify left bottom))
+  )
   (label "PROG_DTR" (at 48.26 46.99 0)
     (effects (font (size 1.27 1.27)) (justify left bottom))
@@
     (effects (font (size 1.27 1.27)) (justify left bottom))
   )
+  (label "WS_OUT" (at 306.07 167.64 180)
+    (effects (font (size 1.27 1.27)) (justify right bottom))
+  )
   (label "PROG_RTS" (at 48.26 44.45 0)
     (effects (font (size 1.27 1.27)) (justify left bottom))
@@
     (effects (font (size 1.27 1.27)) (justify left bottom))
   )
+  (label "LIPO_PRE_MOSFET" (at 30.48 184.15 180)
+    (effects (font (size 1.27 1.27)) (justify right bottom))
+  )
+  (label "WS_OUT" (at 233.68 106.68 180)
+    (effects (font (size 1.27 1.27)) (justify right bottom))
+  )
   (label "PROG_RX" (at 193.04 44.45 0)
     (effects (font (size 1.27 1.27)) (justify left bottom))
@@
     (pin "1")
   )
+  (symbol (lib_id "Connector:TestPoint") (at 243.84 104.14 270) (unit 1)
+    (in_bom yes) (on_board yes)
+    (property "Reference" "TP1" (id 0) (at 242.57 102.87 90)
+      (effects (font (size 1.27 1.27)) (justify left))
+    )
+    (property "Value" "WS_IN" (id 1) (at 248.92 104.14 90)
+      (effects (font (size 1.27 1.27)) (justify left))
+    )
+    (property "Footprint" "TestPoint:TestPoint_Pad_D1.5mm" (id 2) (at 243.84 109.22 0)
+      (effects (font (size 1.27 1.27)) hide)
+    )
+    (property "Datasheet" "~" (id 3) (at 243.84 109.22 0)
+      (effects (font (size 1.27 1.27)) hide)
+    )
+    (pin "1")
+  )
   (symbol (lib_id "Switch:SW_SPDT") (at 124.46 194.31 0) (mirror y) (unit 1)
     (in_bom yes) (on_board yes) (fields_autoplaced)
@@
     (pin "1")
   )
+  (symbol (lib_id "power:+4V") (at 236.22 102.87 0) (unit 1)
+    (in_bom yes) (on_board yes) (fields_autoplaced)
+    (property "Reference" "#PWR0116" (id 0) (at 236.22 106.68 0)
+      (effects (font (size 1.27 1.27)) hide)
+    )
+    (property "Value" "+4V" (id 1) (at 236.22 99.2942 0))
+    (property "Footprint" "" (id 2) (at 236.22 102.87 0)
+      (effects (font (size 1.27 1.27)) hide)
+    )
+    (property "Datasheet" "" (id 3) (at 236.22 102.87 0)
+      (effects (font (size 1.27 1.27)) hide)
+    )
+    (pin "1")
+  )
   (symbol (lib_id "Device:C_Small") (at 71.12 185.42 0) (unit 1)
     (in_bom yes) (on_board yes)
@@
     (pin "1")
   )
+  (symbol (lib_name "GND_29") (lib_id "power:GND") (at 236.22 111.76 0) (unit 1)
+    (in_bom yes) (on_board yes)
+    (property "Reference" "#PWR0121" (id 0) (at 236.22 118.11 0)
+      (effects (font (size 1.27 1.27)) hide)
+    )
+    (property "Value" "GND" (id 1) (at 236.347 116.1542 0)
+      (effects (font (size 1.27 1.27)) hide)
+    )
+    (property "Footprint" "" (id 2) (at 236.22 111.76 0)
+      (effects (font (size 1.27 1.27)) hide)
+    )
+    (property "Datasheet" "" (id 3) (at 236.22 111.76 0)
+      (effects (font (size 1.27 1.27)) hide)
+    )
+    (pin "1")
+  )
   (symbol (lib_id "Switch:SW_Push") (at 140.97 48.26 90) (unit 1)
     (in_bom yes) (on_board yes)
@@
     (pin "1")
   )
+  (symbol (lib_id "Connector:TestPoint") (at 243.84 106.68 270) (unit 1)
+    (in_bom yes) (on_board yes)
+    (property "Reference" "TP2" (id 0) (at 242.57 105.41 90)
+      (effects (font (size 1.27 1.27)) (justify left))
+    )
+    (property "Value" "WS_IN" (id 1) (at 248.92 106.68 90)
+      (effects (font (size 1.27 1.27)) (justify left))
+    )
+    (property "Footprint" "TestPoint:TestPoint_Pad_D1.5mm" (id 2) (at 243.84 111.76 0)
+      (effects (font (size 1.27 1.27)) hide)
+    )
+    (property "Datasheet" "~" (id 3) (at 243.84 111.76 0)
+      (effects (font (size 1.27 1.27)) hide)
+    )
+    (pin "1")
+  )
   (symbol (lib_id "Switch:SW_Push") (at 140.97 95.25 90) (unit 1)
     (in_bom yes) (on_board yes)
@@
     (pin "1")
   )
-  (symbol (lib_id "power:+4V") (at 30.48 184.15 0) (unit 1)
-    (in_bom yes) (on_board yes) (fields_autoplaced)
-    (property "Reference" "#PWR0126" (id 0) (at 30.48 187.96 0)
-      (effects (font (size 1.27 1.27)) hide)
+  (symbol (lib_id "Connector:TestPoint") (at 243.84 109.22 270) (unit 1)
+    (in_bom yes) (on_board yes)
+    (property "Reference" "TP3" (id 0) (at 242.57 107.95 90)
+      (effects (font (size 1.27 1.27)) (justify left))
+    )
+    (property "Value" "WS_IN" (id 1) (at 248.92 109.22 90)
+      (effects (font (size 1.27 1.27)) (justify left))
     )
-    (property "Value" "+4V" (id 1) (at 30.48 180.5742 0))
-    (property "Footprint" "" (id 2) (at 30.48 184.15 0)
+    (property "Footprint" "TestPoint:TestPoint_Pad_D1.5mm" (id 2) (at 243.84 114.3 0)
       (effects (font (size 1.27 1.27)) hide)
     )
-    (property "Datasheet" "" (id 3) (at 30.48 184.15 0)
+    (property "Datasheet" "~" (id 3) (at 243.84 114.3 0)
       (effects (font (size 1.27 1.27)) hide)
     )
@@
       (reference "#PWR0115") (unit 1) (value "GND") (footprint "")
     )
+    (path "/3e3e0542-f3cd-440e-84f4-6519867dd4ed"
+      (reference "#PWR0116") (unit 1) (value "+4V") (footprint "")
+    )
     (path "/ee2df8c9-79b1-4c97-bb0a-01e946fdb061"
       (reference "#PWR0117") (unit 1) (value "GND") (footprint "")
@@
       (reference "#PWR0120") (unit 1) (value "GND") (footprint "")
     )
+    (path "/7a648656-2ab7-4844-920f-9c45863294b3"
+      (reference "#PWR0121") (unit 1) (value "GND") (footprint "")
+    )
     (path "/85ba7e10-919a-43d7-9cec-f5ee16ca38dc"
       (reference "#PWR0122") (unit 1) (value "GND") (footprint "")
@@
       (reference "#PWR0125") (unit 1) (value "GND") (footprint "")
     )
-    (path "/e97d44dd-fb0d-483f-abc9-676ff75c3f6e"
-      (reference "#PWR0126") (unit 1) (value "+4V") (footprint "")
-    )
     (path "/7ead1bfa-520b-4fb1-9dda-ea4b2fdeb7f6"
       (reference "#PWR0127") (unit 1) (value "GND") (footprint "")
@@
       (reference "SW4") (unit 1) (value "RST") (footprint "Button_Switch_SMD:SW_SPST_FSMSM")
     )
+    (path "/262b0fc8-d34c-4e75-8ed6-e8482152a83b"
+      (reference "TP1") (unit 1) (value "WS_IN") (footprint "TestPoint:TestPoint_Pad_D1.5mm")
+    )
+    (path "/bf311c4a-e95a-438d-8bb1-074bb9af12d7"
+      (reference "TP2") (unit 1) (value "WS_IN") (footprint "TestPoint:TestPoint_Pad_D1.5mm")
+    )
+    (path "/e6a3ef32-9a79-4065-b141-669bbcf137ea"
+      (reference "TP3") (unit 1) (value "WS_IN") (footprint "TestPoint:TestPoint_Pad_D1.5mm")
+    )
     (path "/e4753652-aacb-4a7a-aca3-2ada2dbce714"

Commit message: add changes for review
Parts:
- added JP1: TSNS_DIS, Jumper:SolderJumper-2_P1.3mm_Open_TrianglePad1.0x1.5mm, symbol Jumper:SolderJumper_2_Open
- added SW?: B2, Button_Switch_SMD:SW_SPST_TL3342, symbol Switch:SW_Push
- added TH1: NTC_10K, TestPoint:TestPoint_2Pads_Pitch2.54mm_Drill0.8mm, symbol Device:Thermistor_NTC
- R16, R17: footprint Resistor_SMD:R_0201_0603Metric -> Resistor_SMD:R_0603_1608Metric_Pad0.98x0.95mm_HandSolder
Connections:
- net GND: now also SW?.1, TH1.2
- net PROG_DTR: now also Q2.2 (E), R9.1
- net WS_OUT: now also U3.36 (IO22); no longer U3.31 (IO19)
- net at R18.2: now also JP1.1 (A); no longer U5.1 (TS)
- net I2C_RST: no longer names the net of U3.14 (IO12)
- net IN_BUFF_ENA: no longer names the net of U3.16 (IO13)
- net LED_STATUS: no longer names the net of U3.24 (IO2)
- net SCL: no longer names the net of U3.26 (IO4)
- net SDA: no longer names the net of U3.29 (IO5)
- new net: JP1.2 (B), TH1.1, U5.1 (TS)
Other:
- moved on the sheet: C180, F1, H1, H2, H3, H4, J2, Q3, R18, R19, R20, R21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

Commit message: most of routing
Parts:
- added C1, C2, C3, C4: 22uF/handsolder, Capacitor_SMD:C_0805_2012Metric_Pad1.18x1.45mm_HandSolder, symbol Device:C_Small
- added C? (x3): 100n, Capacitor_SMD:C_0201_0603Metric, symbol Device:C_Small
- added R? (x3): 10k, Resistor_SMD:R_0201_0603Metric, symbol Device:R_Small
- C5: value 4.7u -> 22uF/handsolder; footprint Capacitor_SMD:C_0402_1005Metric -> Capacitor_SMD:C_0805_2012Metric_Pad1.18x1.45mm_HandSolder
- gave numbers to parts that had none: 1
Connections:
- net +4V: now also C1.1, C2.1, C3.1, C4.1, R?.1
- net GND: now also C1.2, C2.2, C3.2, C4.2, C?.2, C?.2, C?.2, R?.2
- net at F1.2, R19.1: now also J2.2 (Pin_2); no longer J2.1 (Pin_1)
- net at C180.2, Q3.6 (S2), Q3.7 (S2)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: now also J2.1 (Pin_1); no longer J2.2 (Pin_2)
- net ESP_B3: now reaches SW5.2
- net ESP_B3: now also U3.16 (IO13), C?.1
- net ESP_B2: now reaches SW1.2
- net ESP_B2: now also U3.14 (IO12), C?.1
- net LIPO_VMEAS: now reaches U3.23 (IO15)
- net LIPO_VMEAS: now also C?.1, R?.1, R?.2
- new net: R?.1, R?.2
- no-connect marks 19 -> 20
Other:
- note added: "A couple of tram cap footprints on bottom just in case."
- moved on the sheet: SW1, SW5

Commit message: blah blah routing planes
Parts:
- gave numbers to parts that had none: 6
Changed lines of the file:
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@@
   (symbol (lib_name "GND_25") (lib_id "power:GND") (at 130.81 121.92 0) (unit 1)
     (in_bom yes) (on_board yes)
-    (property "Reference" "#PWR?" (id 0) (at 130.81 128.27 0)
+    (property "Reference" "#PWR0489" (id 0) (at 130.81 128.27 0)
       (effects (font (size 1.27 1.27)) hide)
     )
@@
   (symbol (lib_id "Device:C_Small") (at 130.81 93.98 0) (unit 1)
     (in_bom yes) (on_board yes)
-    (property "Reference" "C?" (id 0) (at 125.73 92.71 0)
+    (property "Reference" "C269" (id 0) (at 125.73 92.71 0)
       (effects (font (size 1.27 1.27)) (justify left))
     )
@@
   (symbol (lib_id "Device:C_Small") (at 130.81 115.57 0) (unit 1)
     (in_bom yes) (on_board yes)
-    (property "Reference" "C?" (id 0) (at 125.73 114.3 0)
+    (property "Reference" "C270" (id 0) (at 125.73 114.3 0)
       (effects (font (size 1.27 1.27)) (justify left))
     )
@@
   (symbol (lib_name "GND_25") (lib_id "power:GND") (at 130.81 100.33 0) (unit 1)
     (in_bom yes) (on_board yes)
-    (property "Reference" "#PWR?" (id 0) (at 130.81 106.68 0)
+    (property "Reference" "#PWR0488" (id 0) (at 130.81 106.68 0)
       (effects (font (size 1.27 1.27)) hide)
     )
@@
   (symbol (lib_id "power:GND") (at 123.19 227.33 0) (mirror y) (unit 1)
     (in_bom yes) (on_board yes) (fields_autoplaced)
-    (property "Reference" "#PWR?" (id 0) (at 123.19 233.68 0)
+    (property "Reference" "#PWR0486" (id 0) (at 123.19 233.68 0)
       (effects (font (size 1.27 1.27)) hide)
     )
@@
   (symbol (lib_id "Device:C_Small") (at 123.19 220.98 0) (unit 1)
     (in_bom yes) (on_board yes)
-    (property "Reference" "C?" (id 0) (at 118.11 219.71 0)
+    (property "Reference" "C271" (id 0) (at 118.11 219.71 0)
       (effects (font (size 1.27 1.27)) (justify left))
     )
@@
   (symbol (lib_id "Device:R_Small") (at 132.08 210.82 0) (mirror y) (unit 1)
     (in_bom yes) (on_board yes)
-    (property "Reference" "R?" (id 0) (at 130.5814 209.6516 0)
+    (property "Reference" "R3" (id 0) (at 130.5814 209.6516 0)
       (effects (font (size 1.27 1.27)) (justify left))
     )
@@
   (symbol (lib_id "power:GND") (at 132.08 234.95 0) (mirror y) (unit 1)
     (in_bom yes) (on_board yes) (fields_autoplaced)
-    (property "Reference" "#PWR?" (id 0) (at 132.08 241.3 0)
+    (property "Reference" "#PWR0428" (id 0) (at 132.08 241.3 0)
       (effects (font (size 1.27 1.27)) hide)
     )
@@
   (symbol (lib_id "Device:R_Small") (at 132.08 220.98 0) (mirror y) (unit 1)
     (in_bom yes) (on_board yes)
-    (property "Reference" "R?" (id 0) (at 130.5814 219.8116 0)
+    (property "Reference" "R6" (id 0) (at 130.5814 219.8116 0)
       (effects (font (size 1.27 1.27)) (justify left))
     )
@@
   (symbol (lib_id "Device:R_Small") (at 132.08 228.6 0) (mirror y) (unit 1)
     (in_bom yes) (on_board yes)
-    (property "Reference" "R?" (id 0) (at 130.5814 227.4316 0)
+    (property "Reference" "R10" (id 0) (at 130.5814 227.4316 0)
       (effects (font (size 1.27 1.27)) (justify left))
     )
@@
       (reference "#PWR0427") (unit 1) (value "+4V") (footprint "")
     )
+    (path "/8e27fc6f-8bb5-43f6-848e-106ee15bb959"
+      (reference "#PWR0428") (unit 1) (value "GND") (footprint "")
+    )
     (path "/eee8c0a8-641e-4924-81da-4e5172896d52/c5504ffa-28ed-4ac8-9bbb-dd9197cdfbdc"
       (reference "#PWR0429") (unit 1) (value "GND") (footprint "")
@@
       (reference "#PWR0485") (unit 1) (value "GND") (footprint "")
     )
+    (path "/7e3c11a5-374e-4a9b-9517-1e539fa6beea"
+      (reference "#PWR0486") (unit 1) (value "GND") (footprint "")
+    )
     (path "/ba681c6f-19d5-423a-a67c-84167cc6e554"
       (reference "#PWR0487") (unit 1) (value "GND") (footprint "")
     )
+    (path "/5a84906d-8287-45ba-8f18-b7c9b99c388e"
+      (reference "#PWR0488") (unit 1) (value "GND") (footprint "")
+    )
+    (path "/2d36ef72-9125-4b7f-9c66-7696e9f2fe5e"
+      (reference "#PWR0489") (unit 1) (value "GND") (footprint "")
+    )
     (path "/55174abd-2342-4b17-bfac-686c8e159bde/53bf4c65-2afd-4326-aa8a-47b57426bd4c"
       (reference "#PWR0492") (unit 1) (value "GND") (footprint "")
@@
       (reference "#PWR0667") (unit 1) (value "GND") (footprint "")
     )
-    (path "/2d36ef72-9125-4b7f-9c66-7696e9f2fe5e"
-      (reference "#PWR?") (unit 1) (value "GND") (footprint "")
-    )
-    (path "/5a84906d-8287-45ba-8f18-b7c9b99c388e"
-      (reference "#PWR?") (unit 1) (value "GND") (footprint "")
-    )
-    (path "/7e3c11a5-374e-4a9b-9517-1e539fa6beea"
-      (reference "#PWR?") (unit 1) (value "GND") (footprint "")
-    )
-    (path "/8e27fc6f-8bb5-43f6-848e-106ee15bb959"
-      (reference "#PWR?") (unit 1) (value "GND") (footprint "")
-    )
     (path "/b43a01de-6c09-412b-8bd2-ed5c96a5aa1f"
       (reference "C1") (unit 1) (value "22uF/handsolder") (footprint "Capacitor_SMD:C_0805_2012Metric_Pad1.18x1.45mm_HandSolder")
@@
     )
     (path "/35bd355e-f3dc-4b38-a1f4-c4e904ac390d"
-      (reference "C?") (unit 1) (value "100n") (footprint "Capacitor_SMD:C_0201_0603Metric")
+      (reference "C269") (unit 1) (value "100n") (footprint "Capacitor_SMD:C_0201_0603Metric")
     )
     (path "/4111770d-7640-4a26-a9d6-2555d69cfb12"
-      (reference "C?") (unit 1) (value "100n") (footprint "Capacitor_SMD:C_0201_0603Metric")
+      (reference "C270") (unit 1) (value "100n") (footprint "Capacitor_SMD:C_0201_0603Metric")
     )
     (path "/7ef312e3-b5f7-48e0-a85b-891c334b6e46"
-      (reference "C?") (unit 1) (value "100n") (footprint "Capacitor_SMD:C_0201_0603Metric")
+      (reference "C271") (unit 1) (value "100n") (footprint "Capacitor_SMD:C_0201_0603Metric")
     )
     (path "/ce3cdc03-45b6-45a7-9791-e23ab3ab8e0e"
@@
       (reference "R2") (unit 1) (value "10k") (footprint "Resistor_SMD:R_0201_0603Metric")
     )
+    (path "/84b7eb65-6c87-48a9-b4db-eeea763c117e"
+      (reference "R3") (unit 1) (value "10k") (footprint "Resistor_SMD:R_0201_0603Metric")
+    )
     (path "/5fa9bf97-4a29-4420-9676-ecb82a4b1452"
       (reference "R4") (unit 1) (value "5.1k") (footprint "Resistor_SMD:R_0201_0603Metric")
@@
       (reference "R5") (unit 1) (value "5.1k") (footprint "Resistor_SMD:R_0201_0603Metric")
     )
+    (path "/cbbe9336-2b0e-41ee-8348-c747cc6425ac"
+      (reference "R6") (unit 1) (value "10k") (footprint "Resistor_SMD:R_0201_0603Metric")
+    )
     (path "/71effdf9-50fc-4eea-8929-f4a022fae592"
       (reference "R7") (unit 1) (value "10k") (footprint "Resistor_SMD:R_0201_0603Metric")
@@
       (reference "R9") (unit 1) (value "10k") (footprint "Resistor_SMD:R_0201_0603Metric")
     )
+    (path "/f722be18-a0dc-4e91-8206-c6b2a1cf8d10"
+      (reference "R10") (unit 1) (value "10k") (footprint "Resistor_SMD:R_0201_0603Metric")
+    )
     (path "/4d59eb96-4933-417d-a01d-a0d35c926e5f"
       (reference "R12") (unit 1) (value "10k") (footprint "Resistor_SMD:R_0201_0603Metric")
@@
       (reference "R21") (unit 1) (value "10k") (footprint "Resistor_SMD:R_0201_0603Metric")
     )
-    (path "/84b7eb65-6c87-48a9-b4db-eeea763c117e"
-      (reference "R?") (unit 1) (value "10k") (footprint "Resistor_SMD:R_0201_0603Metric")
-    )
-    (path "/cbbe9336-2b0e-41ee-8348-c747cc6425ac"
-      (reference "R?") (unit 1) (value "10k") (footprint "Resistor_SMD:R_0201_0603Metric")
-    )
-    (path "/f722be18-a0dc-4e91-8206-c6b2a1cf8d10"
-      (reference "R?") (unit 1) (value "10k") (footprint "Resistor_SMD:R_0201_0603Metric")
-    )
     (path "/bf89ba32-64c5-444b-9eea-ea4b1dc6e76f"
