File: CyberBadge.kicad_sch (KiCad schematic)
At the start: 63 parts, among them J1 USB_C_Receptacle_USB2.0, J2 BAT_CONN, J3 Lichtenprog_conn, Q1 SS8050-G, Q2 SS8050-G, Q3 FS8205A, Q4 AO3401A, SW1 B2, SW2 B1/BOOT, SW3 SW_SPDT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

Commit message: routin sroutin, add bom
Parts:
- D1, D3, D4: footprint LED_SMD:LED_0402_1005Metric -> LED_SMD:LED_0603_1608Metric
Connections:
- net ESP_B2: now also U3.11 (IO26); no longer U3.14 (IO12)
- net ESP_B3: now also U3.10 (IO25); no longer U3.16 (IO13)
Changed lines of the file:
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@@
     (stroke (width 0) (type default) (color 0 0 0 0))
   )
-  (wire (pts (xy 194.31 57.15) (xy 187.96 57.15))
+  (wire (pts (xy 194.31 87.63) (xy 187.96 87.63))
     (stroke (width 0) (type default) (color 0 0 0 0))
   )
@@
     (stroke (width 0) (type default) (color 0 0 0 0))
   )
-  (wire (pts (xy 194.31 59.69) (xy 187.96 59.69))
+  (wire (pts (xy 194.31 85.09) (xy 187.96 85.09))
     (stroke (width 0) (type default) (color 0 0 0 0))
   )
@@
     (effects (font (size 1.27 1.27)) (justify left bottom))
   )
-  (label "ESP_B2" (at 194.31 57.15 0)
+  (label "ESP_B2" (at 194.31 87.63 0)
     (effects (font (size 1.27 1.27)) (justify left bottom))
   )
-  (label "ESP_B3" (at 194.31 59.69 0)
+  (label "ESP_B3" (at 194.31 85.09 0)
     (effects (font (size 1.27 1.27)) (justify left bottom))
   )
@@
       (effects (font (size 1.27 1.27)) (justify right))
     )
-    (property "Footprint" "LED_SMD:LED_0402_1005Metric" (id 2) (at 95.25 175.26 0)
+    (property "Footprint" "LED_SMD:LED_0603_1608Metric" (id 2) (at 95.25 175.26 0)
       (effects (font (size 1.27 1.27)) hide)
     )
@@
       (effects (font (size 1.27 1.27)) (justify right))
     )
-    (property "Footprint" "LED_SMD:LED_0402_1005Metric" (id 2) (at 102.87 175.26 0)
+    (property "Footprint" "LED_SMD:LED_0603_1608Metric" (id 2) (at 102.87 175.26 0)
       (effects (font (size 1.27 1.27)) hide)
     )
@@
       (effects (font (size 1.27 1.27)) (justify right))
     )
-    (property "Footprint" "LED_SMD:LED_0402_1005Metric" (id 2) (at 144.78 212.09 0)
+    (property "Footprint" "LED_SMD:LED_0603_1608Metric" (id 2) (at 144.78 212.09 0)
       (effects (font (size 1.27 1.27)) hide)
     )
@@
     )
     (path "/ce3cdc03-45b6-45a7-9791-e23ab3ab8e0e"
-      (reference "D1") (unit 1) (value "LED") (footprint "LED_SMD:LED_0402_1005Metric")
+      (reference "D1") (unit 1) (value "LED") (footprint "LED_SMD:LED_0603_1608Metric")
     )
     (path "/1942deff-aed8-41b7-8a94-23f87694e4fc"
-      (reference "D3") (unit 1) (value "LED") (footprint "LED_SMD:LED_0402_1005Metric")
+      (reference "D3") (unit 1) (value "LED") (footprint "LED_SMD:LED_0603_1608Metric")
     )
     (path "/3804210c-41cb-449f-87c6-31ac3e0f00b3"
-      (reference "D4") (unit 1) (value "LED") (footprint "LED_SMD:LED_0402_1005Metric")
+      (reference "D4") (unit 1) (value "LED") (footprint "LED_SMD:LED_0603_1608Metric")
     )
     (path "/55174abd-2342-4b17-bfac-686c8e159bde/444f8dc4-e9d2-45d4-a526-33f4fe2d6a8a"
