File: CyberBadge.kicad_sch (KiCad schematic)
At the start: 63 parts, among them J1 USB_C_Receptacle_USB2.0, J2 BAT_CONN, J3 Lichtenprog_conn, Q1 SS8050-G, Q2 SS8050-G, Q3 FS8205A, Q4 AO3401A, SW1 B2, SW2 B1/BOOT, SW3 SW_SPDT, SW4 RST, SW5 B2, U3 ESP32-WROOM-32, U4 SPX3819M5-L-3-3, U5 BQ24073RGT, U6 DW01x

Commit message: schematic cleanup, add PDF and 3D model
Other:
- note added: "A couple of tram cap footprints on bottom just in case. Update: Tests proved those are not required"
- note added: "Rev 1.0.0: Initial release Rev 1.1.0: TODO: Add additional pmos switch directly to battery Add CC line measurement Try to fix buggy DTR/RTS circuit Better battery connector/pads Much larger ESP capacitor tbd."
- note added: "Riset = 890/Itarg Itarg = 0.4A -> Riset=2k Rilim = 1550 / Itarg Iilim = 0.75A -> Rilim=2k"
- note removed: "A couple of tram cap footprints on bottom just in case."
- note removed: "Riset = 890/Itarg Itarg = 0.8A -> Riset=1.1k Itarg = 0.27A -> Riset=3.3k Rilim = 1550 / Itarg Iilim = 1.5A -> Rilim=1.1k"
- note removed: "TODO sprawdzić tranzystory"
- moved on the sheet: C1, C10, C179, C180, C2, C269, C270, C271, C3, C4, C5, C6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

Commit message: add WIP
Parts:
- removed C5: 22uF/handsolder, Capacitor_SMD:C_0805_2012Metric_Pad1.18x1.45mm_HandSolder, symbol Device:C_Small
- removed Q1, Q2: SS8050-G, Package_TO_SOT_SMD:SOT-23, symbol Transistor_BJT:MMBT3904
- removed R12, R9: 10k, Resistor_SMD:R_0201_0603Metric, symbol Device:R_Small
- removed R4, R5: 5.1k, Resistor_SMD:R_0201_0603Metric, symbol Device:R_Small
- removed U3: ESP32-WROOM-32, RF_Module:ESP32-WROOM-32, symbol RF_Module:ESP32-WROOM-32
- added AE?: Antenna_Dipole, RF_Antenna:Texas_SWRA117D_2.4GHz_Right, symbol Device:Antenna_Dipole
- added C? (x2): 3p3, Capacitor_SMD:C_0201_0603Metric, symbol Device:C_Small
- added C? (x5): 100n, Capacitor_SMD:C_0201_0603Metric, symbol Device:C_Small
- added C? (x2): 47uF, Capacitor_SMD:C_0805_2012Metric_Pad1.18x1.45mm_HandSolder, symbol Device:C_Small
- added JP?: PROT_BYP, Jumper:SolderJumper-2_P1.3mm_Open_TrianglePad1.0x1.5mm, symbol Jumper:SolderJumper_2_Open
- added L? (x2): 2n2, symbol Device:L_Small
- added Q?: AO3401A, Package_TO_SOT_SMD:SOT-23, symbol Transistor_FET:AO3401A
- added R? (x2): 200, Resistor_SMD:R_0201_0603Metric, symbol Device:R_Small
- added R? (x2): 5.1k, Resistor_SMD:R_0402_1005Metric, symbol Device:R_Small
- added R? (x2): 100, Resistor_SMD:R_0201_0603Metric, symbol Device:R_Small
- added R?: 0R, Resistor_SMD:R_0201_0603Metric, symbol Device:R_Small
- added U?: USBLC6-2SC6, Package_TO_SOT_SMD:SOT-23-6, symbol Critbit_lib:USBLC6-2SC6
- added U?: LIS3DH, Package_LGA:LGA-16_3x3mm_P0.5mm_LayoutBorder3x5y, symbol Sensor_Motion:LIS3DH
- added U?: ESP32-C3, Package_DFN_QFN:QFN-32-1EP_5x5mm_P0.5mm_EP3.45x3.45mm, symbol Espressif:ESP32-C3
- added Y?: Crystal_GND24, symbol Device:Crystal_GND24
Connections:
- net +3.3V: now also C?.1, C?.1, C?.1, C?.1, C?.1, C?.1, L?.2, U?.11 (VDD3P3_RTC), U?.17 (VDD3P3_CPU), U?.31 (VDDA), U?.32 (VDDA)
- net +4V: no longer R3.1
- net ESP_B2: now also U?.14 (GPIO8)
- net ESP_B3: now also U?.16 (GPIO10)
- net ESP_BOOT: now also U?.15 (GPIO9/BOOT); no longer R7.1
- net ESP_EN: now also U?.7 (CHIP_EN)
- net GND: now also AE?.2, C?.2, C?.2, C?.2, C?.2, C?.2, C?.2, C?.2, C?.2, C?.2, JP?.1 (A), R?.2, R?.2, U?.10 (GND), U?.12 (GND), U?.2 (-), U?.33 (GND), U?.5 (GND), Y?.2, Y?.4
- net LIPO_VMEAS: now also U?.9 (MTMS/GPIO4/ADC1_CH4)
- net PROG_RX: now also R?.2
- net PROG_TX: now also U?.27 (U0RXD/GPIO20)
- net VBUS: now also U?.5 (+)
- net WS_OUT: now also R?.2, U?.10 (MTDI/GPIO5/ADC2_CH0)
- net at J1.B5 (CC2): now also R?.1, R?.2
- net at Q4.1 (G), R1.1, SW3.2 (B): now also Q?.1 (G)
- net at C10.1, F1.1, U5.2 (BAT)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: now also Q?.2 (S)
- net at C180.2, J2.1 (Pin_1), Q3.6 (S2)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: now also JP?.2 (B)
- net at J1.A5 (CC1): now also R?.1, R?.2
- net at J1.A6 (D+): now also J1.B6 (D+), U?.3 (I/O2)
- net at J1.A7 (D-): now also J1.B7 (D-), U?.1 (I/O1)
- new net: R?.1, U?.28 (U0TXD/GPIO21)
- new net: C?.1, L?.1, U?.1 (LNA_IN)
- new net: AE?.1, C?.1, L?.2
- new net: C?.1, L?.1, U?.2 (VDD3P3), U?.3 (VDD3P3)
- new net: Q?.3 (D), R3.1
- new net: U?.29 (XTAL_N), Y?.1
- new net: R?.1, Y?.3
- new net: R?.2, U?.30 (XTAL_P)
- new net CC1: R?.1, U?.6 (GPIO2/ADC1_CH2)
- new net CC2: R?.1, U?.8 (GPIO3/ADC1_CH3)
- new net USBDM: U?.25 (GPIO18/USB_D-), U?.6 (I/O1)
- new net USBDP: U?.26 (GPIO19/USB_D+), U?.4 (I/O2)
- new net WS_2columns/DIN: R?.1
- no-connect marks 20 -> 11
Other:
- note added: "Rev 1.0.0: Initial release Rev 1.1.0: Added additional pmos switch directly to battery TODO: Add CC line measurement Try to fix buggy DTR/RTS circuit Better battery connector/pads Much larger ESP capacitor tbd."
- note removed: "Rev 1.0.0: Initial release Rev 1.1.0: TODO: Add additional pmos switch directly to battery Add CC line measurement Try to fix buggy DTR/RTS circuit Better battery connector/pads Much larger ESP capacitor tbd."
- moved on the sheet: C1, C10, C179, C180, C2, C269, C270, C271, C3, C4, C6, C7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
