File: 1_0/CyberBadge.kicad_pcb (KiCad board)
At the start: 2 copper layers, 112.5 x 41.5 mm, 572 parts, among them J1 USB_C_Receptacle_USB2.0, J2 BAT_CONN, J3 Lichtenprog_conn, Q3 FS8205A, Q4 AO3401A, Q5 AO3401A, SW1 B2, SW2 B1/BOOT, SW3 SW_SPDT, SW4 RST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

Commit message: add files for 2.0
Parts:
- added R12: DNP_0603, Resistor_SMD:R_0603_1608Metric_Pad0.98x0.95mm_HandSolder, B.Cu at (89.9, 103.7)
- added R13: 0R, Resistor_SMD:R_0603_1608Metric_Pad0.98x0.95mm_HandSolder, F.Cu at (82.6, 102.0)
- added R22: DNP_0603, Resistor_SMD:R_0603_1608Metric_Pad0.98x0.95mm_HandSolder, B.Cu at (86.8, 102.5)
- moved C271 0.30 mm to (91.9, 102.6)
- moved C9 0.30 mm to (93.1, 103.0)
- moved R10 0.30 mm to (91.9, 104.4)
- moved R3 0.30 mm to (91.9, 101.7)
- moved R6 0.30 mm to (91.9, 103.5)
- moved R9 0.30 mm to (84.1, 103.6)
- moved R11 0.10 mm to (85.6, 103.6)
Connections:
- Q5 pad 1: unconnected-(Q5-G-Pad1) -> Net-(Q5-G)
- U3 pad 16: unconnected-(U3-IO13-Pad16) -> /LIPO_VMEAS_ENA
Routing:
- net Net-(Q4-G): track 59.4 -> 104.9 mm, vias 2 -> 6
- net /LIPO_VMEAS_ENA: track 0.00 -> 23.4 mm
- net Net-(Q5-G): track 0.00 -> 11.7 mm, vias 0 -> 2
- net /LIPO_VMEAS: track 22.4 -> 18.3 mm
- net Net-(J2-Pin_2): track 26.3 -> 30.0 mm, vias 0 -> 1
- net /PROG_RX: track 37.2 -> 40.3 mm
- net /PROG_TX: track 37.1 -> 40.2 mm
- net +4V: track 605.7 -> 603.7 mm, vias 53 -> 55
- net /ESP_EN: track 49.1 -> 48.4 mm
- net Net-(D17-DOUT): track 5.78 -> 5.98 mm, vias 2 -> 0
