File: 1_0/CyberBadge.kicad_sch (KiCad schematic)
At the start: 56 parts, among them J1 USB_C_Receptacle_USB2.0, J2 BAT_CONN, J3 Lichtenprog_conn, Q3 FS8205A, Q4 AO3401A, Q5 AO3401A, SW1 B2, SW2 B1/BOOT, SW3 SW_SPDT, SW4 RST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

Commit message: add files for 2.0
Parts:
- added R12, R22: DNP_0603, Resistor_SMD:R_0603_1608Metric_Pad0.98x0.95mm_HandSolder, symbol Device:R_Small
- added R13: 0R, Resistor_SMD:R_0603_1608Metric_Pad0.98x0.95mm_HandSolder, symbol Device:R_Small
Connections:
- net at F1.2, J2.2 (Pin_2), Q5.2 (S)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: now also R12.2
- net at Q4.1 (G), R1.1, SW3.2 (B): now also R13.1
- net at Q5.1 (G): now also R12.1, R13.2, R22.1
- net LIPO_VMEAS_ENA: now reaches U3.16 (IO13)
- net LIPO_VMEAS_ENA: now also R22.2
Changed lines of the file:
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@@
   (junction (at 302.26 64.77) (diameter 0) (color 0 0 0 0)
   )
+  (junction (at 80.01 198.12) (diameter 0) (color 0 0 0 0)
+  )
   (junction (at 281.94 64.77) (diameter 0) (color 0 0 0 0)
   )
@@
   )
   (junction (at 322.58 137.16) (diameter 0) (color 0 0 0 0)
+  )
+  (junction (at 53.34 203.2) (diameter 0) (color 0 0 0 0)
+  )
+  (junction (at 60.96 203.2) (diameter 0) (color 0 0 0 0)
+  )
+  (junction (at 128.27 173.99) (diameter 0) (color 0 0 0 0)
   )
   (junction (at 218.44 175.26) (diameter 0) (color 0 0 0 0)
@@
     (stroke (width 0) (type default))
   )
-  (wire (pts (xy 128.27 163.83) (xy 128.27 187.96))
+  (wire (pts (xy 128.27 163.83) (xy 128.27 173.99))
     (stroke (width 0) (type default))
   )
@@
     (stroke (width 0) (type default))
   )
+  (wire (pts (xy 128.27 173.99) (xy 128.27 187.96))
+    (stroke (width 0) (type default))
+  )
   (wire (pts (xy 80.01 212.09) (xy 80.01 208.28))
     (stroke (width 0) (type default))
@@
     (stroke (width 0) (type default))
   )
-  (wire (pts (xy 62.23 203.2) (xy 72.39 203.2))
-    (stroke (width 0) (type default))
-  )
   (wire (pts (xy 48.895 93.98) (xy 51.435 93.98))
     (stroke (width 0) (type default))
@@
     (stroke (width 0) (type default))
   )
+  (wire (pts (xy 48.26 203.2) (xy 53.34 203.2))
+    (stroke (width 0) (type default))
+  )
   (wire (pts (xy 83.82 260.35) (xy 83.82 255.27))
     (stroke (width 0) (type default))
@@
     (stroke (width 0) (type default))
   )
+  (wire (pts (xy 53.34 194.31) (xy 53.34 198.12))
+    (stroke (width 0) (type default))
+  )
   (wire (pts (xy 302.26 87.63) (xy 302.26 91.44))
     (stroke (width 0) (type default))
@@
     (stroke (width 0) (type default))
   )
+  (wire (pts (xy 101.6 173.99) (xy 101.6 194.31))
+    (stroke (width 0) (type default))
+  )
   (wire (pts (xy 186.69 40.64) (xy 191.77 40.64))
     (stroke (width 0) (type default))
@@
     (stroke (width 0) (type default))
   )
+  (wire (pts (xy 39.37 203.2) (xy 43.18 203.2))
+    (stroke (width 0) (type default))
+  )
   (wire (pts (xy 129.54 81.28) (xy 143.51 81.28))
     (stroke (width 0) (type default))
@@
     (stroke (width 0) (type default))
   )
+  (wire (pts (xy 53.34 203.2) (xy 60.96 203.2))
+    (stroke (width 0) (type default))
+  )
   (wire (pts (xy 161.29 175.26) (xy 161.29 177.8))
     (stroke (width 0) (type default))
@@
     (stroke (width 0) (type default))
   )
+  (wire (pts (xy 60.96 203.2) (xy 72.39 203.2))
+    (stroke (width 0) (type default))
+  )
   (wire (pts (xy 261.62 64.77) (xy 261.62 68.58))
     (stroke (width 0) (type default))
@@
     (stroke (width 0) (type default))
   )
+  (wire (pts (xy 186.69 50.8) (xy 207.01 50.8))
+    (stroke (width 0) (type default))
+  )
   (wire (pts (xy 186.69 35.56) (xy 191.77 35.56))
     (stroke (width 0) (type default))
@@
     (stroke (width 0) (type default))
   )
+  (wire (pts (xy 60.96 198.12) (xy 80.01 198.12))
+    (stroke (width 0) (type default))
+  )
+  (wire (pts (xy 128.27 173.99) (xy 101.6 173.99))
+    (stroke (width 0) (type default))
+  )
   (wire (pts (xy 56.515 93.98) (xy 59.055 93.98))
     (stroke (width 0) (type default))
@@
   )
   (wire (pts (xy 86.36 143.51) (xy 86.36 139.7))
+    (stroke (width 0) (type default))
+  )
+  (wire (pts (xy 101.6 194.31) (xy 53.34 194.31))
     (stroke (width 0) (type default))
   )
@@
     (effects (font (size 1.27 1.27)) (justify left bottom))
   )
+  (label "LIPO_VMEAS_ENA" (at 39.37 203.2 180) (fields_autoplaced)
+    (effects (font (size 1.27 1.27)) (justify right bottom))
+  )
   (label "PROG_DTR" (at 43.815 38.1 0) (fields_autoplaced)
     (effects (font (size 1.27 1.27)) (justify left bottom))
@@
     (effects (font (size 1.27 1.27)) (justify right bottom))
   )
+  (label "LIPO_VMEAS_ENA" (at 207.01 50.8 0) (fields_autoplaced)
+    (effects (font (size 1.27 1.27)) (justify left bottom))
+  )
   (label "ESP_B2" (at 143.51 81.28 0) (fields_autoplaced)
     (effects (font (size 1.27 1.27)) (justify left bottom))
@@
         (path "/0335a998-9fbe-49b9-adca-aa3d90d195f2"
           (reference "R5") (unit 1)
+        )
+      )
+    )
+  )
+  (symbol (lib_id "Device:R_Small") (at 60.96 200.66 0) (mirror x) (unit 1)
+    (in_bom yes) (on_board yes) (dnp no)
+    (property "Reference" "R12" (at 63.5 199.39 0)
+      (effects (font (size 1.27 1.27)))
+    )
+    (property "Value" "DNP_0603" (at 64.135 201.295 0)
+      (effects (font (size 1.27 1.27)))
+    )
+    (property "Footprint" "Resistor_SMD:R_0603_1608Metric_Pad0.98x0.95mm_HandSolder" (at 60.96 200.66 0)
+      (effects (font (size 1.27 1.27)) hide)
+    )
+    (property "Datasheet" "~" (at 60.96 200.66 0)
+      (effects (font (size 1.27 1.27)) hide)
+    )
+    (property "LCSC" "C25117" (at 60.96 200.66 0)
+      (effects (font (size 1.27 1.27)) hide)
+    )
+    (pin "1")
+    (pin "2")
+    (instances
+      (project "CyberBadge"
+        (path "/0335a998-9fbe-49b9-adca-aa3d90d195f2"
+          (reference "R12") (unit 1)
         )
       )
@@
     )
   )
+  (symbol (lib_id "Device:R_Small") (at 53.34 200.66 0) (mirror y) (unit 1)
+    (in_bom yes) (on_board yes) (dnp no)
+    (property "Reference" "R13" (at 57.15 199.39 0)
+      (effects (font (size 1.27 1.27)))
+    )
+    (property "Value" "0R" (at 55.88 201.93 0)
+      (effects (font (size 1.27 1.27)))
+    )
+    (property "Footprint" "Resistor_SMD:R_0603_1608Metric_Pad0.98x0.95mm_HandSolder" (at 53.34 200.66 0)
+      (effects (font (size 1.27 1.27)) hide)
+    )
+    (property "Datasheet" "~" (at 53.34 200.66 0)
+      (effects (font (size 1.27 1.27)) hide)
+    )
+    (property "LCSC" "C25117" (at 53.34 200.66 0)
+      (effects (font (size 1.27 1.27)) hide)
+    )
+    (pin "1")
+    (pin "2")
+    (instances
+      (project "CyberBadge"
+        (path "/0335a998-9fbe-49b9-adca-aa3d90d195f2"
+          (reference "R13") (unit 1)
+        )
+      )
+    )
+  )
   (symbol (lib_id "power:GND") (at 71.12 231.14 0) (mirror y) (unit 1)
     (in_bom yes) (on_board yes) (dnp no) (fields_autoplaced)
@@
         )
       )
+    )
+  )
+  (symbol (lib_id "Device:R_Small") (at 45.72 203.2 270) (mirror x) (unit 1)
+    (in_bom yes) (on_board yes) (dnp no)
+    (property "Reference" "R22" (at 45.72 200.66 90)
+      (effects (font (size 1.27 1.27)))
+    )
+    (property "Value" "DNP_0603" (at 45.72 205.74 90)
+      (effects (font (size 1.27 1.27)))
+    )
+    (property "Footprint" "Resistor_SMD:R_0603_1608Metric_Pad0.98x0.95mm_HandSolder" (at 45.72 203.2 0)
+      (effects (font (size 1.27 1.27)) hide)
+    )
+    (property "Datasheet" "~" (at 45.72 203.2 0)
+      (effects (font (size 1.27 1.27)) hide)
+    )
+    (property "LCSC" "C25117" (at 45.72 203.2 0)
+      (effects (font (size 1.27 1.27)) hide)
+    )
+    (pin "1")
+    (pin "2")
+    (instances
+      (project "CyberBadge"
+        (path "/0335a998-9fbe-49b9-adca-aa3d90d195f2"
+          (reference "R22") (unit 1)
+        )
+      )
