File: 2_0/ledboad/PMOS.kicad_sch (KiCad schematic)
At the start: 1 part, among them Q11 CJX3139K

Commit message: before oder
Parts:
- Q11: LCSC (none) -> C504144; LCSC Part C504144 -> (none)
Changed lines of the file:
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@@
 			)
 		)
-		(property "LCSC Part" "C504144"
+		(property "LCSC Part" ""
 			(at 118.11 82.55 0)
 			(effects
 				(font
+					(size 1.27 1.27)
+				)
+				(hide yes)
+			)
+		)
+		(property "LCSC" "C504144"
+			(at 118.11 67.31 0)
+			(effects
+				(font
