File: 2_0/ledboad/ledboad.kicad_sch (KiCad schematic)
At the start: 333 parts, among them J1 Conn_02x05_Odd_Even, Q4 AO3401A, SW1 RST, U1 STM32G070CBTx, U2 XC6206PxxxMR, Y1 2016/DNP

Commit message: commit before rescheme
Parts:
- removed C1, C3: 100n, Capacitor_SMD:C_0402_1005Metric, symbol Device:C_Small
- removed C2, C4: 470n, Capacitor_SMD:C_0402_1005Metric, symbol Device:C_Small
- removed C7, C8: 10p/DNP, Capacitor_SMD:C_0402_1005Metric, symbol Device:C_Small
- removed D1: LED_RGBA, Critbit_lib:0606, symbol Device:LED_RABG
- removed J1: Conn_02x05_Odd_Even, Critbit_lib:YXT-BB10-10S, symbol Connector_Generic:Conn_02x05_Odd_Even
- removed R15, R16, R17: 10k, Resistor_SMD:R_0402_1005Metric, symbol Device:R_Small
- removed SW1: RST, Button_Switch_SMD:SW_SPST_FSMSM, symbol Switch:SW_Push
- removed TP1, TP10, TP11, TP12, TP13, TP14, TP15, TP16, TP17, TP18, TP19, TP2, TP20, TP21, TP22, TP23, TP24, TP25, TP26, TP27, TP28, TP29, TP3, TP30, TP31, TP32, TP4, TP5, TP6, TP7, TP8, TP9: TP, TestPoint:TestPoint_Pad_D1.0mm, symbol Connector:TestPoint
- removed U1: STM32G070CBTx, Package_QFP:LQFP-48_7x7mm_P0.5mm, symbol MCU_ST_STM32G0:STM32G070CBTx
- removed U2: XC6206PxxxMR, Package_TO_SOT_SMD:SOT-23-3, symbol Regulator_Linear:XC6206PxxxMR
- removed Y1: 2016/DNP, Crystal:Crystal_SMD_2016-4Pin_2.0x1.6mm, symbol Device:Crystal_GND24
- added J1: USB_C_Receptacle_USB2.0, Connector_USB:USB_C_Receptacle_HRO_TYPE-C-31-M-12, symbol Connector:USB_C_Receptacle_USB2.0
- added R18, R19: 5.1k, Resistor_SMD:R_0201_0603Metric, symbol Device:R_Small
- added U2: 74HC138PW,118, easyeda2kicad:SSOP-16_L6.2-W5.3-P0.65-LS7.8-BL, symbol easyeda2kicad:74HC138PW,118
- added U3: ~, Critbit_lib:pilkbrain, symbol Critbit_lib:pilkbrain
Connections:
- net COL_B0: now also RU5.5 (O0); no longer RU1.7 (O2)
- net COL_B1: now also RU5.6 (O1); no longer RU1.10 (O5)
- net COL_B10: now also RU5.15 (O10); no longer RU5.5 (O0)
- net COL_B11: now also RU5.16 (O11); no longer RU5.8 (O3)
- net COL_B12: now also RU5.17 (O12); no longer RU5.11 (O6)
- net COL_B13: now also RU5.18 (O13); no longer RU5.14 (O9)
- net COL_B14: now also RU5.19 (O14); no longer RU5.17 (O12)
- net COL_B16: now also RU6.5 (O0); no longer RU2.7 (O2)
- net COL_B17: now also RU6.6 (O1); no longer RU2.10 (O5)
- net COL_B18: now also RU6.7 (O2); no longer RU2.13 (O8)
- net COL_B19: now also RU6.8 (O3); no longer RU2.16 (O11)
- net COL_B2: now also RU5.7 (O2); no longer RU1.13 (O8)
- net COL_B20: now also RU6.9 (O4); no longer RU2.19 (O14)
- net COL_B21: now also RU6.10 (O5); no longer RU4.6 (O1)
- net COL_B22: now also RU6.11 (O6); no longer RU4.9 (O4)
- net COL_B23: now also RU6.12 (O7); no longer RU4.12 (O7)
- net COL_B24: now also RU6.13 (O8); no longer RU4.15 (O10)
- net COL_B25: now also RU6.14 (O9); no longer RU4.18 (O13)
- net COL_B26: now also RU6.15 (O10); no longer RU6.5 (O0)
- net COL_B27: now also RU6.16 (O11); no longer RU6.8 (O3)
- net COL_B28: now also RU6.17 (O12); no longer RU6.11 (O6)
- net COL_B29: now also RU6.18 (O13); no longer RU6.14 (O9)
- net COL_B3: now also RU5.8 (O3); no longer RU1.16 (O11)
- net COL_B30: now also RU6.19 (O14); no longer RU6.17 (O12)
- net COL_B4: now also RU5.9 (O4); no longer RU1.19 (O14)
- net COL_B5: now also RU5.10 (O5); no longer RU3.6 (O1)
- net COL_B6: now also RU5.11 (O6); no longer RU3.9 (O4)
- net COL_B7: now also RU5.12 (O7); no longer RU3.12 (O7)
- net COL_B8: now also RU5.13 (O8); no longer RU3.15 (O10)
- net COL_B9: now also RU5.14 (O9); no longer RU3.18 (O13)
- net COL_G0: now also RU3.5 (O0); no longer RU1.6 (O1)
- net COL_G1: now also RU3.6 (O1); no longer RU1.9 (O4)
- net COL_G10: now also RU3.15 (O10); no longer RU3.20 (O15)
- net COL_G11: now also RU3.16 (O11); no longer RU5.7 (O2)
- net COL_G12: now also RU3.17 (O12); no longer RU5.10 (O5)
- net COL_G13: now also RU3.18 (O13); no longer RU5.13 (O8)
- net COL_G14: now also RU3.19 (O14); no longer RU5.16 (O11)
- net COL_G15: now also RU3.20 (O15); no longer RU5.19 (O14)
- net COL_G16: now also RU4.5 (O0); no longer RU2.6 (O1)
- net COL_G17: now also RU4.6 (O1); no longer RU2.9 (O4)
- net COL_G18: now also RU4.7 (O2); no longer RU2.12 (O7)
- net COL_G19: now also RU4.8 (O3); no longer RU2.15 (O10)
- net COL_G2: now also RU3.7 (O2); no longer RU1.12 (O7)
- net COL_G20: now also RU4.9 (O4); no longer RU2.18 (O13)
- net COL_G21: now also RU4.10 (O5); no longer RU4.5 (O0)
- net COL_G22: now also RU4.11 (O6); no longer RU4.8 (O3)
- net COL_G23: now also RU4.12 (O7); no longer RU4.11 (O6)
- net COL_G24: now also RU4.13 (O8); no longer RU4.14 (O9)
- net COL_G25: now also RU4.14 (O9); no longer RU4.17 (O12)
- net COL_G26: now also RU4.15 (O10); no longer RU4.20 (O15)
- net COL_G27: now also RU4.16 (O11); no longer RU6.7 (O2)
- net COL_G28: now also RU4.17 (O12); no longer RU6.10 (O5)
- net COL_G29: now also RU4.18 (O13); no longer RU6.13 (O8)
- net COL_G3: now also RU3.8 (O3); no longer RU1.15 (O10)
- net COL_G30: now also RU4.19 (O14); no longer RU6.16 (O11)
- net COL_G31: now also RU4.20 (O15); no longer RU6.19 (O14)
- net COL_G4: now also RU3.9 (O4); no longer RU1.18 (O13)
- net COL_G5: now also RU3.10 (O5); no longer RU3.5 (O0)
- net COL_G6: now also RU3.11 (O6); no longer RU3.8 (O3)
- net COL_G7: now also RU3.12 (O7); no longer RU3.11 (O6)
- net COL_G8: now also RU3.13 (O8); no longer RU3.14 (O9)
- net COL_G9: now also RU3.14 (O9); no longer RU3.17 (O12)
- net COL_R1: now also RU1.6 (O1); no longer RU1.8 (O3)
- net COL_R10: now also RU1.15 (O10); no longer RU3.19 (O14)
- net COL_R11: now also RU1.16 (O11); no longer RU5.6 (O1)
- net COL_R12: now also RU1.17 (O12); no longer RU5.9 (O4)
- net COL_R13: now also RU1.18 (O13); no longer RU5.12 (O7)
- net COL_R14: now also RU1.19 (O14); no longer RU5.15 (O10)
- net COL_R15: now also RU1.20 (O15); no longer RU5.18 (O13)
- net COL_R17: now also RU2.6 (O1); no longer RU2.8 (O3)
- net COL_R18: now also RU2.7 (O2); no longer RU2.11 (O6)
- net COL_R19: now also RU2.8 (O3); no longer RU2.14 (O9)
- net COL_R2: now also RU1.7 (O2); no longer RU1.11 (O6)
- net COL_R20: now also RU2.9 (O4); no longer RU2.17 (O12)
- net COL_R21: now also RU2.10 (O5); no longer RU2.20 (O15)
- net COL_R22: now also RU2.11 (O6); no longer RU4.7 (O2)
- net COL_R23: now also RU2.12 (O7); no longer RU4.10 (O5)
- net COL_R24: now also RU2.13 (O8); no longer RU4.13 (O8)
- net COL_R25: now also RU2.14 (O9); no longer RU4.16 (O11)
- net COL_R26: now also RU2.15 (O10); no longer RU4.19 (O14)
- net COL_R27: now also RU2.16 (O11); no longer RU6.6 (O1)
- net COL_R28: now also RU2.17 (O12); no longer RU6.9 (O4)
- net COL_R29: now also RU2.18 (O13); no longer RU6.12 (O7)
- net COL_R3: now also RU1.8 (O3); no longer RU1.14 (O9)
- net COL_R30: now also RU2.19 (O14); no longer RU6.15 (O10)
- net COL_R31: now also RU2.20 (O15); no longer RU6.18 (O13)
- net COL_R4: now also RU1.9 (O4); no longer RU1.17 (O12)
- net COL_R5: now also RU1.10 (O5); no longer RU1.20 (O15)
- net COL_R6: now also RU1.11 (O6); no longer RU3.7 (O2)
- net COL_R7: now also RU1.12 (O7); no longer RU3.10 (O5)
- net COL_R8: now also RU1.13 (O8); no longer RU3.13 (O8)
- net COL_R9: now also RU1.14 (O9); no longer RU3.16 (O11)
- net GND: now also J1.A1 (GND), J1.A12 (GND), J1.B1 (GND), J1.B12 (GND), J1.S1 (SHIELD), R18.2, R19.2, U2.8 (GND), U3.G (GND)
- net LAT: now also U3.5
- net OE: now also U3.6
- net ROW_0_CTRL: now also U2.15 (~{Y0})
- net ROW_1_CTRL: now also U2.14 (~{Y1})
- net ROW_2_CTRL: now also U2.13 (~{Y2})
- net ROW_3_CTRL: now also U2.12 (~{Y3})
- net ROW_4_CTRL: now also U2.11 (~{Y4})
- net ROW_5_CTRL: now also U2.10 (~{Y5})
- net ROW_6_CTRL: now also U2.9 (~{Y6})
- net ROW_7_CTRL: now also U2.7 (~{Y7})
- net SCLK: now also U3.10
- net VDD: now also U2.16 (VCC), U3.4V (LIPO_OUT)
- net DAT0 renamed DAT_R
- net DAT_R: now also U3.7
- net DAT1: no longer names the net of RU1.22 (SDO)
- net DAT1: now also RU2.2 (SDI); no longer RU3.2 (SDI)
- net DAT2: no longer names the net of RU3.22 (SDO)
- net DAT2: now also RU4.2 (SDI); no longer RU5.2 (SDI)
- net DAT3: no longer names the net of RU5.22 (SDO)
- net DAT3: now also RU6.2 (SDI); no longer RU2.2 (SDI)
- net DAT4: no longer names the net of RU2.22 (SDO)
- net DAT4: no longer RU4.2 (SDI)
- net DAT5: no longer names the net of RU4.22 (SDO)
- net DAT5: no longer RU6.2 (SDI)
- net DAT6: no longer names the net of RU6.22 (SDO)
- new net: J1.A5 (CC1), R18.1
- new net: J1.B5 (CC2), R19.1
- new net DAT_B: RU5.2 (SDI), U3.9
- new net DAT_G: RU3.2 (SDI), U3.8
- new net DM: J1.A7 (D-), J1.B7 (D-), U3.DM (USB_DM)
- new net DP: J1.A6 (D+), J1.B6 (D+), U3.DP (USB_DP)
- new net MATRIX_A: U2.1 (A0), U3.2
- new net MATRIX_B: U2.2 (A1), U3.3
- new net MATRIX_C: U2.3 (A2), U3.4
- new net VBUS: J1.A4 (VBUS), J1.A9 (VBUS), J1.B4 (VBUS), J1.B9 (VBUS), U3.5V (5V_IN)
- no-connect marks 0 -> 18
Other:
- note removed: "VDD cause layout"
- note removed: "https://www.lcsc.com/product-detail/Microcontroller-Units-MCUs-MPUs-SOCs_STMicroelectronics-STM32G070CBT6_C529338.html"
- moved on the sheet: Q4, R1, R2, R3, R4, R5, R6, R7, R8

Commit message: rescheme, reroute
Parts:
- removed C10: 470n, Capacitor_SMD:C_0402_1005Metric, symbol Device:C_Small
- removed Q4 (x8): AO3401A, Package_TO_SOT_SMD:SOT-23, symbol Transistor_FET:AO3401A
- removed R1, R2, R3, R4, R5, R6, R7, R8: 10k, Resistor_SMD:R_0402_1005Metric, symbol Device:R_Small
- removed U3: ~, Critbit_lib:pilkbrain, symbol Critbit_lib:pilkbrain
- added C1, C2, C3, C4, C6: 470n, Capacitor_SMD:C_0402_1005Metric, symbol Device:C_Small
- added R15, R16, R17, R20, R21, R22, R23, R24: 10k, Resistor_SMD:R_0402_1005Metric, symbol Device:R_Small
- added SW2: TS-1088-AR02016, easyeda2kicad:SW-SMD_L3.9-W3.0-P4.45, symbol easyeda2kicad:TS-1088-AR02016
Connections:
- net COL_B0: now also RU6.20 (O15); no longer RU5.5 (O0)
- net COL_B1: now also RU6.19 (O14); no longer RU5.6 (O1)
- net COL_B10: now also RU6.10 (O5); no longer RU5.15 (O10)
- net COL_B11: now also RU6.9 (O4); no longer RU5.16 (O11)
- net COL_B12: now also RU6.8 (O3); no longer RU5.17 (O12)
- net COL_B13: now also RU6.7 (O2); no longer RU5.18 (O13)
- net COL_B14: now also RU6.6 (O1); no longer RU5.19 (O14)
- net COL_B15: now also RU6.5 (O0); no longer RU5.20 (O15)
- net COL_B16: now also RU5.20 (O15); no longer RU6.5 (O0)
- net COL_B17: now also RU5.19 (O14); no longer RU6.6 (O1)
- net COL_B18: now also RU5.18 (O13); no longer RU6.7 (O2)
- net COL_B19: now also RU5.17 (O12); no longer RU6.8 (O3)
- net COL_B2: now also RU6.18 (O13); no longer RU5.7 (O2)
- net COL_B20: now also RU5.16 (O11); no longer RU6.9 (O4)
- net COL_B21: now also RU5.15 (O10); no longer RU6.10 (O5)
- net COL_B22: now also RU5.14 (O9); no longer RU6.11 (O6)
- net COL_B23: now also RU5.13 (O8); no longer RU6.12 (O7)
- net COL_B24: now also RU5.12 (O7); no longer RU6.13 (O8)
- net COL_B25: now also RU5.11 (O6); no longer RU6.14 (O9)
- net COL_B26: now also RU5.10 (O5); no longer RU6.15 (O10)
- net COL_B27: now also RU5.9 (O4); no longer RU6.16 (O11)
- net COL_B28: now also RU5.8 (O3); no longer RU6.17 (O12)
- net COL_B29: now also RU5.7 (O2); no longer RU6.18 (O13)
- net COL_B3: now also RU6.17 (O12); no longer RU5.8 (O3)
- net COL_B30: now also RU5.6 (O1); no longer RU6.19 (O14)
- net COL_B31: now also RU5.5 (O0); no longer RU6.20 (O15)
- net COL_B4: now also RU6.16 (O11); no longer RU5.9 (O4)
- net COL_B5: now also RU6.15 (O10); no longer RU5.10 (O5)
- net COL_B6: now also RU6.14 (O9); no longer RU5.11 (O6)
- net COL_B7: now also RU6.13 (O8); no longer RU5.12 (O7)
- net COL_B8: now also RU6.12 (O7); no longer RU5.13 (O8)
- net COL_B9: now also RU6.11 (O6); no longer RU5.14 (O9)
- net COL_G0: now also RU4.20 (O15); no longer RU3.5 (O0)
- net COL_G1: now also RU4.19 (O14); no longer RU3.6 (O1)
- net COL_G10: now also RU4.10 (O5); no longer RU3.15 (O10)
- net COL_G11: now also RU4.9 (O4); no longer RU3.16 (O11)
- net COL_G12: now also RU4.8 (O3); no longer RU3.17 (O12)
- net COL_G13: now also RU4.7 (O2); no longer RU3.18 (O13)
- net COL_G14: now also RU4.6 (O1); no longer RU3.19 (O14)
- net COL_G15: now also RU4.5 (O0); no longer RU3.20 (O15)
- net COL_G16: now also RU3.20 (O15); no longer RU4.5 (O0)
- net COL_G17: now also RU3.19 (O14); no longer RU4.6 (O1)
- net COL_G18: now also RU3.18 (O13); no longer RU4.7 (O2)
- net COL_G19: now also RU3.17 (O12); no longer RU4.8 (O3)
- net COL_G2: now also RU4.18 (O13); no longer RU3.7 (O2)
- net COL_G20: now also RU3.16 (O11); no longer RU4.9 (O4)
- net COL_G21: now also RU3.15 (O10); no longer RU4.10 (O5)
- net COL_G22: now also RU3.14 (O9); no longer RU4.11 (O6)
- net COL_G23: now also RU3.13 (O8); no longer RU4.12 (O7)
- net COL_G24: now also RU3.12 (O7); no longer RU4.13 (O8)
- net COL_G25: now also RU3.11 (O6); no longer RU4.14 (O9)
- net COL_G26: now also RU3.10 (O5); no longer RU4.15 (O10)
- net COL_G27: now also RU3.9 (O4); no longer RU4.16 (O11)
- net COL_G28: now also RU3.8 (O3); no longer RU4.17 (O12)
- net COL_G29: now also RU3.7 (O2); no longer RU4.18 (O13)
- net COL_G3: now also RU4.17 (O12); no longer RU3.8 (O3)
- net COL_G30: now also RU3.6 (O1); no longer RU4.19 (O14)
- net COL_G31: now also RU3.5 (O0); no longer RU4.20 (O15)
- net COL_G4: now also RU4.16 (O11); no longer RU3.9 (O4)
- net COL_G5: now also RU4.15 (O10); no longer RU3.10 (O5)
- net COL_G6: now also RU4.14 (O9); no longer RU3.11 (O6)
- net COL_G7: now also RU4.13 (O8); no longer RU3.12 (O7)
- net COL_G8: now also RU4.12 (O7); no longer RU3.13 (O8)
- net COL_G9: now also RU4.11 (O6); no longer RU3.14 (O9)
- net COL_R0: now also RU2.20 (O15); no longer RU1.5 (O0)
- net COL_R1: now also RU2.19 (O14); no longer RU1.6 (O1)
- net COL_R10: now also RU2.10 (O5); no longer RU1.15 (O10)
- net COL_R11: now also RU2.9 (O4); no longer RU1.16 (O11)
- net COL_R12: now also RU2.8 (O3); no longer RU1.17 (O12)
- net COL_R13: now also RU2.7 (O2); no longer RU1.18 (O13)
- net COL_R14: now also RU2.6 (O1); no longer RU1.19 (O14)
- net COL_R15: now also RU2.5 (O0); no longer RU1.20 (O15)
- net COL_R16: now also RU1.20 (O15); no longer RU2.5 (O0)
- net COL_R17: now also RU1.19 (O14); no longer RU2.6 (O1)
- net COL_R18: now also RU1.18 (O13); no longer RU2.7 (O2)
- net COL_R19: now also RU1.17 (O12); no longer RU2.8 (O3)
- net COL_R2: now also RU2.18 (O13); no longer RU1.7 (O2)
- net COL_R20: now also RU1.16 (O11); no longer RU2.9 (O4)
- net COL_R21: now also RU1.15 (O10); no longer RU2.10 (O5)
- net COL_R22: now also RU1.14 (O9); no longer RU2.11 (O6)
- net COL_R23: now also RU1.13 (O8); no longer RU2.12 (O7)
- net COL_R24: now also RU1.12 (O7); no longer RU2.13 (O8)
- net COL_R25: now also RU1.11 (O6); no longer RU2.14 (O9)
- net COL_R26: now also RU1.10 (O5); no longer RU2.15 (O10)
- net COL_R27: now also RU1.9 (O4); no longer RU2.16 (O11)
- net COL_R28: now also RU1.8 (O3); no longer RU2.17 (O12)
- net COL_R29: now also RU1.7 (O2); no longer RU2.18 (O13)
- net COL_R3: now also RU2.17 (O12); no longer RU1.8 (O3)
- net COL_R30: now also RU1.6 (O1); no longer RU2.19 (O14)
- net COL_R31: now also RU1.5 (O0); no longer RU2.20 (O15)
- net COL_R4: now also RU2.16 (O11); no longer RU1.9 (O4)
- net COL_R5: now also RU2.15 (O10); no longer RU1.10 (O5)
- net COL_R6: now also RU2.14 (O9); no longer RU1.11 (O6)
- net COL_R7: now also RU2.13 (O8); no longer RU1.12 (O7)
- net COL_R8: now also RU2.12 (O7); no longer RU1.13 (O8)
- net COL_R9: now also RU2.11 (O6); no longer RU1.14 (O9)
- net GND: now also C1.2, C2.2, C3.2, C4.2, C6.2
- net ROW_0_CTRL: now also R15.2
- net ROW_1_CTRL: now also R16.2
- net ROW_2_CTRL: now also R17.2
- net ROW_3_CTRL: now also R20.2
- net ROW_4_CTRL: now also R21.2
- net ROW_5_CTRL: now also R22.2
- net ROW_6_CTRL: now also R23.2
- net ROW_7_CTRL: now also R24.2
- net VDD: now also C1.1, C2.1, C3.1, C4.1, C6.1, R15.1, R16.1, R17.1, R20.1, R21.1, R22.1, R23.1, R24.1
Other:
- added sheet PMOS (PMOS.kicad_sch)
- added sheet PMOS1 (PMOS.kicad_sch)
- added sheet PMOS2 (PMOS.kicad_sch)
- added sheet PMOS3 (PMOS.kicad_sch)
- added sheet PMOS4 (PMOS.kicad_sch)
- added sheet PMOS5 (PMOS.kicad_sch)
- added sheet PMOS6 (PMOS.kicad_sch)
- added sheet PMOS7 (PMOS.kicad_sch)
- moved on the sheet: R10, R11, R13, R9, RU1, RU2, RU3, RU5

Commit message: work on ledboard
Parts:
- added C7: 470n, Capacitor_SMD:C_0402_1005Metric, symbol Device:C_Small
- added SW1, SW3: TS-1088-AR02016, easyeda2kicad:SW-SMD_L3.9-W3.0-P4.45, symbol easyeda2kicad:TS-1088-AR02016
- added U1: ~, Critbit_lib:pilkbrain2, symbol Critbit_lib:pilkbrain2
- R18, R19: footprint Resistor_SMD:R_0201_0603Metric -> Resistor_SMD:R_0402_1005Metric
Connections:
- net COL_B0: now also RU6.5 (O0); no longer RU6.20 (O15)
- net COL_B1: now also RU6.6 (O1); no longer RU6.19 (O14)
- net COL_B10: now also RU6.15 (O10); no longer RU6.10 (O5)
- net COL_B11: now also RU6.16 (O11); no longer RU6.9 (O4)
- net COL_B12: now also RU6.17 (O12); no longer RU6.8 (O3)
- net COL_B13: now also RU6.18 (O13); no longer RU6.7 (O2)
- net COL_B14: now also RU6.19 (O14); no longer RU6.6 (O1)
- net COL_B15: now also RU6.20 (O15); no longer RU6.5 (O0)
- net COL_B16: now also RU5.5 (O0); no longer RU5.20 (O15)
- net COL_B17: now also RU5.6 (O1); no longer RU5.19 (O14)
- net COL_B18: now also RU5.7 (O2); no longer RU5.18 (O13)
- net COL_B19: now also RU5.8 (O3); no longer RU5.17 (O12)
- net COL_B2: now also RU6.7 (O2); no longer RU6.18 (O13)
- net COL_B20: now also RU5.9 (O4); no longer RU5.16 (O11)
- net COL_B21: now also RU5.10 (O5); no longer RU5.15 (O10)
- net COL_B22: now also RU5.11 (O6); no longer RU5.14 (O9)
- net COL_B23: now also RU5.12 (O7); no longer RU5.13 (O8)
- net COL_B24: now also RU5.13 (O8); no longer RU5.12 (O7)
- net COL_B25: now also RU5.14 (O9); no longer RU5.11 (O6)
- net COL_B26: now also RU5.15 (O10); no longer RU5.10 (O5)
- net COL_B27: now also RU5.16 (O11); no longer RU5.9 (O4)
- net COL_B28: now also RU5.17 (O12); no longer RU5.8 (O3)
- net COL_B29: now also RU5.18 (O13); no longer RU5.7 (O2)
- net COL_B3: now also RU6.8 (O3); no longer RU6.17 (O12)
- net COL_B30: now also RU5.19 (O14); no longer RU5.6 (O1)
- net COL_B31: now also RU5.20 (O15); no longer RU5.5 (O0)
- net COL_B4: now also RU6.9 (O4); no longer RU6.16 (O11)
- net COL_B5: now also RU6.10 (O5); no longer RU6.15 (O10)
- net COL_B6: now also RU6.11 (O6); no longer RU6.14 (O9)
- net COL_B7: now also RU6.12 (O7); no longer RU6.13 (O8)
- net COL_B8: now also RU6.13 (O8); no longer RU6.12 (O7)
- net COL_B9: now also RU6.14 (O9); no longer RU6.11 (O6)
- net COL_G0: now also RU4.5 (O0); no longer RU4.20 (O15)
- net COL_G1: now also RU4.6 (O1); no longer RU4.19 (O14)
- net COL_G10: now also RU4.15 (O10); no longer RU4.10 (O5)
- net COL_G11: now also RU4.16 (O11); no longer RU4.9 (O4)
- net COL_G12: now also RU4.17 (O12); no longer RU4.8 (O3)
- net COL_G13: now also RU4.18 (O13); no longer RU4.7 (O2)
- net COL_G14: now also RU4.19 (O14); no longer RU4.6 (O1)
- net COL_G15: now also RU4.20 (O15); no longer RU4.5 (O0)
- net COL_G16: now also RU3.5 (O0); no longer RU3.20 (O15)
- net COL_G17: now also RU3.6 (O1); no longer RU3.19 (O14)
- net COL_G18: now also RU3.7 (O2); no longer RU3.18 (O13)
- net COL_G19: now also RU3.8 (O3); no longer RU3.17 (O12)
- net COL_G2: now also RU4.7 (O2); no longer RU4.18 (O13)
- net COL_G20: now also RU3.9 (O4); no longer RU3.16 (O11)
- net COL_G21: now also RU3.10 (O5); no longer RU3.15 (O10)
- net COL_G22: now also RU3.11 (O6); no longer RU3.14 (O9)
- net COL_G23: now also RU3.12 (O7); no longer RU3.13 (O8)
- net COL_G24: now also RU3.13 (O8); no longer RU3.12 (O7)
- net COL_G25: now also RU3.14 (O9); no longer RU3.11 (O6)
- net COL_G26: now also RU3.15 (O10); no longer RU3.10 (O5)
- net COL_G27: now also RU3.16 (O11); no longer RU3.9 (O4)
- net COL_G28: now also RU3.17 (O12); no longer RU3.8 (O3)
- net COL_G29: now also RU3.18 (O13); no longer RU3.7 (O2)
- net COL_G3: now also RU4.8 (O3); no longer RU4.17 (O12)
- net COL_G30: now also RU3.19 (O14); no longer RU3.6 (O1)
- net COL_G31: now also RU3.20 (O15); no longer RU3.5 (O0)
- net COL_G4: now also RU4.9 (O4); no longer RU4.16 (O11)
- net COL_G5: now also RU4.10 (O5); no longer RU4.15 (O10)
- net COL_G6: now also RU4.11 (O6); no longer RU4.14 (O9)
- net COL_G7: now also RU4.12 (O7); no longer RU4.13 (O8)
- net COL_G8: now also RU4.13 (O8); no longer RU4.12 (O7)
- net COL_G9: now also RU4.14 (O9); no longer RU4.11 (O6)
- net COL_R0: now also RU2.5 (O0); no longer RU2.20 (O15)
- net COL_R1: now also RU2.6 (O1); no longer RU2.19 (O14)
- net COL_R10: now also RU2.15 (O10); no longer RU2.10 (O5)
- net COL_R11: now also RU2.16 (O11); no longer RU2.9 (O4)
- net COL_R12: now also RU2.17 (O12); no longer RU2.8 (O3)
- net COL_R13: now also RU2.18 (O13); no longer RU2.7 (O2)
- net COL_R14: now also RU2.19 (O14); no longer RU2.6 (O1)
- net COL_R15: now also RU2.20 (O15); no longer RU2.5 (O0)
- net COL_R16: now also RU1.5 (O0); no longer RU1.20 (O15)
- net COL_R17: now also RU1.6 (O1); no longer RU1.19 (O14)
- net COL_R18: now also RU1.7 (O2); no longer RU1.18 (O13)
- net COL_R19: now also RU1.8 (O3); no longer RU1.17 (O12)
- net COL_R2: now also RU2.7 (O2); no longer RU2.18 (O13)
- net COL_R20: now also RU1.9 (O4); no longer RU1.16 (O11)
- net COL_R21: now also RU1.10 (O5); no longer RU1.15 (O10)
- net COL_R22: now also RU1.11 (O6); no longer RU1.14 (O9)
- net COL_R23: now also RU1.12 (O7); no longer RU1.13 (O8)
- net COL_R24: now also RU1.13 (O8); no longer RU1.12 (O7)
- net COL_R25: now also RU1.14 (O9); no longer RU1.11 (O6)
- net COL_R26: now also RU1.15 (O10); no longer RU1.10 (O5)
- net COL_R27: now also RU1.16 (O11); no longer RU1.9 (O4)
- net COL_R28: now also RU1.17 (O12); no longer RU1.8 (O3)
- net COL_R29: now also RU1.18 (O13); no longer RU1.7 (O2)
- net COL_R3: now also RU2.8 (O3); no longer RU2.17 (O12)
- net COL_R30: now also RU1.19 (O14); no longer RU1.6 (O1)
- net COL_R31: now also RU1.20 (O15); no longer RU1.5 (O0)
- net COL_R4: now also RU2.9 (O4); no longer RU2.16 (O11)
- net COL_R5: now also RU2.10 (O5); no longer RU2.15 (O10)
- net COL_R6: now also RU2.11 (O6); no longer RU2.14 (O9)
- net COL_R7: now also RU2.12 (O7); no longer RU2.13 (O8)
- net COL_R8: now also RU2.13 (O8); no longer RU2.12 (O7)
- net COL_R9: now also RU2.14 (O9); no longer RU2.11 (O6)
- net DAT_B: now also RU6.2 (SDI), U1.5; no longer RU5.2 (SDI)
- net DAT_G: now also RU4.2 (SDI), U1.4; no longer RU3.2 (SDI)
- net DAT_R: now also RU2.2 (SDI), U1.3; no longer RU1.2 (SDI)
- net DM: now also U1.DM (USB_DM)
- net DP: now also U1.DP (USB_DP)
- net GND: now also C7.2, U1.G (GND)
- net LAT: now also U1.1
- net MATRIX_A: now also U1.6
- net MATRIX_B: now also U1.7
- net MATRIX_C: now also U1.8
- net OE: now also U1.2
- net SCLK: now also U1.D (WS2812_DAT)
- net VBUS: now also U1.5V (5V_IN)
- net VDD: now also C7.1, U1.4V (LIPO_OUT)
- net at RU3.22 (SDO): no longer RU4.2 (SDI)
- net at RU4.22 (SDO): now also RU3.2 (SDI)
- net at RU1.22 (SDO): no longer RU2.2 (SDI)
- net at RU5.22 (SDO): no longer RU6.2 (SDI)
- net at RU6.22 (SDO): now also RU5.2 (SDI)
- net at RU2.22 (SDO): now also RU1.2 (SDI)
- no-connect marks 18 -> 13
Other:
- moved on the sheet: C1, C2, C3, C4, C5, C6, D0_1, D0_2, D0_3, D0_4, D0_5, D0_6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

Commit message: before oder
Parts:
- added C10, C8, C9: 470n, Capacitor_SMD:C_0402_1005Metric, symbol Device:C_Small
- added JP1, JP2, JP3: SB, Jumper:SolderJumper-2_P1.3mm_Bridged_RoundedPad1.0x1.5mm, symbol Jumper:SolderJumper_2_Bridged
- C1, C2, C3, C4, C5, C6, C7: LCSC (none) -> C52923
- D0_1, D0_2, D0_3, D0_4, D0_5, D0_6, D0_7, D0_8, D10_1, D10_2, D10_3, D10_4, D10_5, D10_6, D10_7, D10_8, D11_1, D11_2, D11_3, D11_4, D11_5, D11_6, D11_7, D11_8, D12_1, D12_2, D12_3, D12_4, D12_5, D12_6, D12_7, D12_8, D13_1, D13_2, D13_3, D13_4, D13_5, D13_6, D13_7, D13_8, D14_1, D14_2, D14_3, D14_4, D14_5, D14_6, D14_7, D14_8, D15_1, D15_2, D15_3, D15_4, D15_5, D15_6, D15_7, D15_8, D16_1, D16_2, D16_3, D16_4, D16_5, D16_6, D16_7, D16_8, D17_1, D17_2, D17_3, D17_4, D17_5, D17_6, D17_7, D17_8, D18_1, D18_2, D18_3, D18_4, D18_5, D18_6, D18_7, D18_8, D19_1, D19_2, D19_3, D19_4, D19_5, D19_6, D19_7, D19_8, D1_1, D1_2, D1_3, D1_4, D1_5, D1_6, D1_7, D1_8, D20_1, D20_2, D20_3, D20_4, D20_5, D20_6, D20_7, D20_8, D21_1, D21_2, D21_3, D21_4, D21_5, D21_6, D21_7, D21_8, D22_1, D22_2, D22_3, D22_4, D22_5, D22_6, D22_7, D22_8, D23_1, D23_2, D23_3, D23_4, D23_5, D23_6, D23_7, D23_8, D24_1, D24_2, D24_3, D24_4, D24_5, D24_6, D24_7, D24_8, D25_1, D25_2, D25_3, D25_4, D25_5, D25_6, D25_7, D25_8, D26_1, D26_2, D26_3, D26_4, D26_5, D26_6, D26_7, D26_8, D27_1, D27_2, D27_3, D27_4, D27_5, D27_6, D27_7, D27_8, D28_1, D28_2, D28_3, D28_4, D28_5, D28_6, D28_7, D28_8, D29_1, D29_2, D29_3, D29_4, D29_5, D29_6, D29_7, D29_8, D2_1, D2_2, D2_3, D2_4, D2_5, D2_6, D2_7, D2_8, D30_1, D30_2, D30_3, D30_4, D30_5, D30_6, D30_7, D30_8, D31_1, D31_2, D31_3, D31_4, D31_5, D31_6, D31_7, D31_8, D3_1, D3_2, D3_3, D3_4, D3_5, D3_6, D3_7, D3_8, D4_1, D4_2, D4_3, D4_4, D4_5, D4_6, D4_7, D4_8, D5_1, D5_2, D5_3, D5_4, D5_5, D5_6, D5_7, D5_8, D6_1, D6_2, D6_3, D6_4, D6_5, D6_6, D6_7, D6_8, D7_1, D7_2, D7_3, D7_4, D7_5, D7_6, D7_7, D7_8, D8_1, D8_2, D8_3, D8_4, D8_5, D8_6, D8_7, D8_8, D9_1, D9_2, D9_3, D9_4, D9_5, D9_6, D9_7, D9_8: LCSC (none) -> C2874115
- R10, R11, R12, R13, R14, R9: LCSC (none) -> C25123
- R15, R16, R17, R20, R21, R22, R23, R24: LCSC (none) -> C25744
- R18, R19: LCSC C25117 -> C25905
- RU1, RU2, RU3, RU4, RU5, RU6: LCSC (none) -> C121618
- SW1, SW2, SW3: LCSC (none) -> C720477; LCSC Part C720477 -> (none)
- U2: LCSC (none) -> C47455; LCSC Part C47455 -> (none)
Connections:
- net GND: now also SW1.2, SW2.2, SW3.2, C10.2, C8.2, C9.2, JP1.2 (B), JP2.2 (B)
- net VDD: now also JP3.2 (B)
- net at U2.4 (~{E1}): now also JP1.1 (A)
- net at U2.5 (~{E2}): now also JP2.1 (A)
- net at U2.6 (E3): now also JP3.1 (A)
- net B2: now reaches SW2.1
- net B2: now also U1.SCL, C8.1
- net at SW3.1: now also C10.1
- net B1: now reaches SW1.1
- net B1: now also U1.SDA, C9.1
- no-connect marks 13 -> 12
Other:
- moved on the sheet: SW1, SW2, SW3
